File: out/hub/slimevr-i2spi-hub.kicad_sch (KiCad schematic)
At the start: 33 parts, among them J1 RJ45-CHAIN, J2 LiPo, J3 USB-C, SW1 BOOT, U1 ESP32-C5-WROOM-1, U2 ICM-45686, U3 QMC6309, U4 AP2112K-3.3, U5 MCP73831

Commit message: Fix the node ATtiny412 pinout; regenerate stale outputs
gen/boards.py wired the node's ATtiny412 as if pin 2 were UPDI and pin 6 the strobe. The
SOIC-8 part is 1 VCC, 2 PA6, 3 PA7, 4 PA1, 5 PA2, 6 PA0/UPDI, 7 PA3, 8 GND (KiCad's
ATtiny202-SS symbol, which ATtiny412-SS extends), so six of eight pins were on the wrong
pads: strobe, chip select, both chain I2C lines, UPDI and the sensor power gate.

- ATTINY412 now declares pin_functions, and gen/check_node_pins.py checks the board's
  nets against both that map and the ports the node firmware drives. It runs in
  verify.sh, needs no KiCad, and reports 6 wrong on the old mapping.
- verify.py follows (extends ...) in KiCad symbols; ATtiny412-SS previously read as "not
  installed", so its pins could never be checked.
- mksch.py resolves a part's candidate symbols against the KiCad library instead of
  writing the "|"-joined list into the schematic, which KiCad cannot load. Without a
  library it stops rather than pick a MOSFET symbol with an unknown pin order.
- out/ regenerated for the documented 18-point build (5 hubs, 8 nodes). The committed
  files were from the single preset and predated the datasheet re-pin of the hub.
- docs/BOARD-SPECS.md hub and node pin tables now follow gen/boards.py, with module and
  SOIC pin numbers; README says where each pinout comes from.

Hub ESP32-C5 pins were cross-checked against the vendored Espressif symbol: all match.
Checked with KiCad 8.0.9 symbol libraries; footprint libraries were not installed.

Co-Authored-By: Claude Opus 5.5 <noreply@anthropic.com>
Claude-Session: https://claude.ai/code/session_01Sb26stwPJiCMHhrBWZ2D9q
Parts:
- added J4: UART, Connector_JST:JST_PH_S2B-PH-SM4-TB_1x02-1MP_P2.00mm_Horizontal, symbol Connector:Conn_01x02_Pin
- added R18: 10k, Resistor_SMD:R_0402_1005Metric, symbol Device:R
- R16: Note IO2 is a strapping pin: hold it defined -> MTMS strapping pin: hold it defined
- R17: Note IO7 is a strapping pin: hold it defined -> MTDI strapping pin (SDIO edge): hold it defined

Commit message: Check pins against pads, fix the USB-C symbol, add CI, record licences
verify.py:
- Every symbol pin must have a pad on the part's footprint, and every pin a board wires
  must exist on its symbol. This caught the USB-C part: the full USB_C_Receptacle symbol
  has SuperSpeed pins the 16-pad HRO TYPE-C-31-M-12 has no pads for. It now uses
  USB_C_Receptacle_USB2.0_16P (USB_C_Receptacle_USB2.0 in KiCad 7), which matches pad
  for pad.
- Unit sub-symbols are matched exactly: looking up Device:R also collected
  R_Network08's pins, which could pass or fail a pin map on another part's pins.
- Hidden pins (bare `hide` before or after the length, or KiCad 9's (hide yes)) are
  read. Stacked power pins are usually hidden; the ESP32-C5's EPAD grounds and USB-C's
  VBUS/GND pairs were invisible to the checker before.
- KiCad 10's one-file-per-symbol libraries (*.kicad_symdir) are read alongside the
  single-file libraries KiCad 7-9 install.

With KiCad 8.0.9 symbols and footprints: 15 parts, 0 problems; pin-order guard 4/4.

CI runs verify.sh with Ubuntu's KiCad symbol and footprint packages installed.

lib/vendor: Espressif's libraries are CC-BY-SA 4.0 with KiCad's design exception; the
licence text is now alongside them. The Mumo library's licence is unknown and recorded
as such in PROVENANCE.md; only its QMC6309 symbol and footprint are used.

Co-Authored-By: Claude Opus 5.5 <noreply@anthropic.com>
Claude-Session: https://claude.ai/code/session_01Sb26stwPJiCMHhrBWZ2D9q
Parts:
- removed J3: USB-C, Connector_USB:USB_C_Receptacle_HRO_TYPE-C-31-M-12, symbol Connector:USB_C_Receptacle
- added J3: USB-C, Connector_USB:USB_C_Receptacle_HRO_TYPE-C-31-M-12, symbol Connector:USB_C_Receptacle_USB2.0_16P
Changed lines of the file:
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@@
     (effects (font (size 1.27 1.27)) (justify left))
   )
-  (symbol (lib_id "Connector:USB_C_Receptacle") (at 165.10 304.80 0) (unit 1)
+  (symbol (lib_id "Connector:USB_C_Receptacle_USB2.0_16P") (at 165.10 304.80 0) (unit 1)
     (in_bom yes) (on_board yes)
     (property "Reference" "J3" (at 165.10 292.10 0)
