File: out/node/slimevr-i2spi-node.kicad_sch (KiCad schematic)
At the start: 16 parts, among them J1 RJ45-IN, J2 RJ45-OUT, Q1 DMG2305UX, U1 ATtiny412, U2 ICM-45686, U3 QMC6309

Commit message: Fix the node ATtiny412 pinout; regenerate stale outputs
gen/boards.py wired the node's ATtiny412 as if pin 2 were UPDI and pin 6 the strobe. The
SOIC-8 part is 1 VCC, 2 PA6, 3 PA7, 4 PA1, 5 PA2, 6 PA0/UPDI, 7 PA3, 8 GND (KiCad's
ATtiny202-SS symbol, which ATtiny412-SS extends), so six of eight pins were on the wrong
pads: strobe, chip select, both chain I2C lines, UPDI and the sensor power gate.

- ATTINY412 now declares pin_functions, and gen/check_node_pins.py checks the board's
  nets against both that map and the ports the node firmware drives. It runs in
  verify.sh, needs no KiCad, and reports 6 wrong on the old mapping.
- verify.py follows (extends ...) in KiCad symbols; ATtiny412-SS previously read as "not
  installed", so its pins could never be checked.
- mksch.py resolves a part's candidate symbols against the KiCad library instead of
  writing the "|"-joined list into the schematic, which KiCad cannot load. Without a
  library it stops rather than pick a MOSFET symbol with an unknown pin order.
- out/ regenerated for the documented 18-point build (5 hubs, 8 nodes). The committed
  files were from the single preset and predated the datasheet re-pin of the hub.
- docs/BOARD-SPECS.md hub and node pin tables now follow gen/boards.py, with module and
  SOIC pin numbers; README says where each pinout comes from.

Hub ESP32-C5 pins were cross-checked against the vendored Espressif symbol: all match.
Checked with KiCad 8.0.9 symbol libraries; footprint libraries were not installed.

Co-Authored-By: Claude Opus 5.5 <noreply@anthropic.com>
Claude-Session: https://claude.ai/code/session_01Sb26stwPJiCMHhrBWZ2D9q
Parts:
- U3: Note on the IMU AUX1 bus, not the chain -> 4-pad WLCSP on the IMU AUX1 bus, not the chain
Changed lines of the file:
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@@
     (title "SlimeVR I2SPI sensor node")
     (company "SlimeVR I2SPI")
-    (comment 1 "Generated by hardware/gen/mksch.py - do not hand-edit, regenerate")
+    (comment 1 "Generated by gen/mksch.py - do not hand-edit, regenerate")
     (comment 2 "ATtiny412 + gated ICM-45686 + QMC6309, two RJ45 jacks")
   )
@@
     (effects (font (size 1.27 1.27)) (justify left))
   )
-  (global_label "UPDI" (shape bidirectional) (at 182.88 30.48 0)
-    (effects (font (size 1.27 1.27)) (justify left))
-  )
-  (global_label "CHAIN_SDA" (shape bidirectional) (at 182.88 33.02 0)
-    (effects (font (size 1.27 1.27)) (justify left))
-  )
-  (global_label "CHAIN_SCL" (shape bidirectional) (at 182.88 35.56 0)
-    (effects (font (size 1.27 1.27)) (justify left))
-  )
-  (global_label "SENSOR_PWR_G" (shape bidirectional) (at 182.88 38.10 0)
-    (effects (font (size 1.27 1.27)) (justify left))
-  )
-  (global_label "CS_STROBE" (shape bidirectional) (at 182.88 40.64 0)
-    (effects (font (size 1.27 1.27)) (justify left))
-  )
-  (global_label "CS_IMU" (shape bidirectional) (at 182.88 43.18 0)
+  (global_label "CS_STROBE" (shape bidirectional) (at 182.88 30.48 0)
+    (effects (font (size 1.27 1.27)) (justify left))
+  )
+  (global_label "CS_IMU" (shape bidirectional) (at 182.88 33.02 0)
+    (effects (font (size 1.27 1.27)) (justify left))
+  )
+  (global_label "CHAIN_SDA" (shape bidirectional) (at 182.88 35.56 0)
+    (effects (font (size 1.27 1.27)) (justify left))
+  )
+  (global_label "CHAIN_SCL" (shape bidirectional) (at 182.88 38.10 0)
+    (effects (font (size 1.27 1.27)) (justify left))
+  )
+  (global_label "UPDI" (shape bidirectional) (at 182.88 40.64 0)
+    (effects (font (size 1.27 1.27)) (justify left))
+  )
+  (global_label "SENSOR_PWR_G" (shape bidirectional) (at 182.88 43.18 0)
     (effects (font (size 1.27 1.27)) (justify left))
   )
@@
       (effects (font (size 1.27 1.27)) hide))
   )
-  (global_label "AUX_SCL" (shape bidirectional) (at 119.38 66.04 0)
-    (effects (font (size 1.27 1.27)) (justify left))
-  )
-  (global_label "CS_IMU" (shape bidirectional) (at 119.38 68.58 0)
-    (effects (font (size 1.27 1.27)) (justify left))
-  )
-  (global_label "SPI_SCK" (shape bidirectional) (at 119.38 71.12 0)
-    (effects (font (size 1.27 1.27)) (justify left))
-  )
-  (global_label "SPI_MOSI" (shape bidirectional) (at 119.38 73.66 0)
-    (effects (font (size 1.27 1.27)) (justify left))
-  )
-  (global_label "GND" (shape bidirectional) (at 119.38 78.74 0)
+  (global_label "SPI_MISO" (shape bidirectional) (at 119.38 66.04 0)
+    (effects (font (size 1.27 1.27)) (justify left))
+  )
+  (global_label "CS_IMU" (shape bidirectional) (at 119.38 73.66 0)
+    (effects (font (size 1.27 1.27)) (justify left))
+  )
+  (global_label "SPI_SCK" (shape bidirectional) (at 119.38 76.20 0)
+    (effects (font (size 1.27 1.27)) (justify left))
+  )
+  (global_label "SPI_MOSI" (shape bidirectional) (at 119.38 78.74 0)
     (effects (font (size 1.27 1.27)) (justify left))
   )
@@
     (effects (font (size 1.27 1.27)) (justify left))
   )
+  (global_label "AUX_SCL" (shape bidirectional) (at 119.38 83.82 0)
+    (effects (font (size 1.27 1.27)) (justify left))
+  )
   (global_label "VSENSOR" (shape bidirectional) (at 119.38 88.90 0)
     (effects (font (size 1.27 1.27)) (justify left))
@@
     (effects (font (size 1.27 1.27)) (justify left))
   )
-  (global_label "SPI_MISO" (shape bidirectional) (at 119.38 99.06 0)
-    (effects (font (size 1.27 1.27)) (justify left))
-  )
   (symbol (lib_id "Mumo:QMC6309") (at 165.10 76.20 0) (unit 1)
     (in_bom yes) (on_board yes)
@@
     (property "Footprint" "Mumo:QMC6309" (at 165.10 76.20 0)
       (effects (font (size 1.27 1.27)) hide))
-    (property "Note" "on the IMU AUX1 bus, not the chain" (at 165.10 76.20 0)
-      (effects (font (size 1.27 1.27)) hide))
-  )
-  (global_label "AUX_SCL" (shape bidirectional) (at 182.88 66.04 0)
-    (effects (font (size 1.27 1.27)) (justify left))
-  )
-  (global_label "GND" (shape bidirectional) (at 182.88 68.58 0)
-    (effects (font (size 1.27 1.27)) (justify left))
-  )
-  (global_label "AUX_SDA" (shape bidirectional) (at 182.88 71.12 0)
-    (effects (font (size 1.27 1.27)) (justify left))
-  )
-  (global_label "VSENSOR" (shape bidirectional) (at 182.88 73.66 0)
-    (effects (font (size 1.27 1.27)) (justify left))
-  )
+    (property "Note" "4-pad WLCSP on the IMU AUX1 bus, not the chain" (at 165.10 76.20 0)
+      (effects (font (size 1.27 1.27)) hide))
+  )
+  (global_label "GND" (shape bidirectional) (at 182.88 66.04 0)
+    (effects (font (size 1.27 1.27)) (justify left))
+  )
+  (global_label "AUX_SCL" (shape bidirectional) (at 182.88 68.58 0)
+    (effects (font (size 1.27 1.27)) (justify left))
+  )
+  (global_label "VSENSOR" (shape bidirectional) (at 182.88 71.12 0)
+    (effects (font (size 1.27 1.27)) (justify left))
+  )
+  (global_label "AUX_SDA" (shape bidirectional) (at 182.88 73.66 0)
+    (effects (font (size 1.27 1.27)) (justify left))
+  )
